Commit message: Add files via upload

File: data/hand.urdf (robot description, URDF)
Before this commit: robot hand, 15 links, 14 joints
Links:
- added link index-finger-lower, mass 1.0; collision cylinder length=0.1 radius=0.025; visual cylinder length=0.1 radius=0.025
- added link middle-finger-lower, mass 1.0; collision cylinder length=0.1 radius=0.025; visual cylinder length=0.1 radius=0.025
- added link pinky-finger-lower, mass 1.0; collision cylinder length=0.1 radius=0.025; visual cylinder length=0.1 radius=0.025
- added link ring-finger-lower, mass 1.0; collision cylinder length=0.1 radius=0.025; visual cylinder length=0.1 radius=0.025
- added link thumb-base, mass 1.0; collision cylinder length=0.1 radius=0.025; visual cylinder length=0.1 radius=0.025
- added link thumb-lower, mass 1.0; collision cylinder length=0.1 radius=0.025; visual cylinder length=0.1 radius=0.025
- added link thumb-top, mass 1.0; collision cylinder length=0.1 radius=0.025; visual cylinder length=0.1 radius=0.025
- link index-finger-base: geometry collision sphere radius=0.025; visual sphere radius=0.025
- link index-finger-top: geometry collision cylinder length=0.1 radius=0.025; visual cylinder length=0.075 radius=0.025
- link middle-finger-base: geometry collision sphere radius=0.025; visual sphere radius=0.025
- link palm: geometry collision box size=0.35 0.2 0.05; visual box size=0.275 0.2 0.05
- link pinky-finger-base: geometry collision sphere radius=0.025; visual sphere radius=0.025
- link pinky-finger-top: geometry collision cylinder length=0.1 radius=0.025; visual cylinder length=0.075 radius=0.025
- link ring-finger-base: geometry collision sphere radius=0.025; visual sphere radius=0.025
Joints:
- removed joint index-finger-mcp
- removed joint middle-finger-mcp
- removed joint pinky-finger-mcp
- removed joint ring-finger-mcp
- added joint index-finger-mcp1: type revolute, parent palm, child index-finger-base, origin xyz=-0.075 0 0 rpy=0 0 0, axis 0 0 1, limit lower=0 upper=0.52 effort=1000 velocity=1
- added joint index-finger-mcp2: type revolute, parent index-finger-base, child index-finger-lower, origin xyz=0 0 0 rpy=0 0 0, axis 1 0 0, limit lower=-1.57 upper=0 effort=1000 velocity=1
- added joint middle-finger-mcp1: type revolute, parent palm, child middle-finger-base, origin xyz=0 0 0 rpy=0 0 0, axis 0 0 1, limit lower=0 upper=0.26 effort=1000 velocity=1
- added joint middle-finger-mcp2: type revolute, parent middle-finger-base, child middle-finger-lower, origin xyz=0 0 0 rpy=0 0 0, axis 1 0 0, limit lower=-1.57 upper=0 effort=1000 velocity=1
- added joint pinky-finger-mcp1: type revolute, parent palm, child pinky-finger-base, origin xyz=0.15 0 0 rpy=0 0 0, axis 0 0 1, limit lower=-0.52 upper=0 effort=1000 velocity=1
- added joint pinky-finger-mcp2: type revolute, parent pinky-finger-base, child pinky-finger-lower, origin xyz=0 0 0 rpy=0 0 0, axis 1 0 0, limit lower=-1.57 upper=0 effort=1000 velocity=1
- added joint ring-finger-mcp1: type revolute, parent palm, child ring-finger-base, origin xyz=0.075 0 0 rpy=0 0 0, axis 0 0 1, limit lower=-0.26 upper=0 effort=1000 velocity=1
- added joint ring-finger-mcp2: type revolute, parent ring-finger-base, child ring-finger-lower, origin xyz=0 0 0 rpy=0 0 0, axis 1 0 0, limit lower=-1.57 upper=0 effort=1000 velocity=1
- added joint thumb-cmc: type revolute, parent palm-base, child thumb-base, origin xyz=-0.15 -0.2 0 rpy=0 0 0, axis 1 0 0, limit lower=-1.57 upper=0 effort=1000 velocity=1
- added joint thumb-ip: type revolute, parent thumb-lower, child thumb-top, origin xyz=0 0.1 0 rpy=0 0 0, axis 0 0 1, limit lower=-1.57 upper=0 effort=1000 velocity=1
- added joint thumb-mcp: type revolute, parent thumb-base, child thumb-lower, origin xyz=0 0.1 0 rpy=0 0 0, axis 0 0 1, limit lower=-1.57 upper=0 effort=1000 velocity=1
- joint index-finger-pip: parent index-finger-base -> index-finger-lower
- joint middle-finger-pip: parent middle-finger-base -> middle-finger-lower
- joint pinky-finger-pip: parent pinky-finger-base -> pinky-finger-lower
- joint ring-finger-pip: parent ring-finger-base -> ring-finger-lower
